File: MainBoardV2/MainBoardV2.kicad_pcb (KiCad board)
At the start: 2 copper layers, 98 x 87.9 mm, 50 parts, among them J1 Conn_01x02, J10 Conn_01x04, J11 Conn_01x02, J12 Conn_01x03, J13 Conn_01x03, J14 Conn_01x03, J15 Conn_01x03, J16 Conn_01x02, J17 Conn_01x02, J18 Conn_01x03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

Commit message: hOLDUP
Routing:
- net EN: track 152.9 -> 151.5 mm
Changed lines of the file:
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@@
   (segment (start 64.9224 141.1224) (end 68.32872 144.52872) (width 1.5) (layer "F.Cu") (net 8))
   (segment (start 47.6504 127.7112) (end 46.5836 127.7112) (width 1.5) (layer "F.Cu") (net 8))
+  (segment (start 47.6504 151.3332) (end 45.9232 151.3332) (width 1.5) (layer "F.Cu") (net 8))
   (segment (start 46.482 107.2896) (end 55.1688 107.2896) (width 1.5) (layer "F.Cu") (net 8))
-  (segment (start 45.212 151.3332) (end 42.3164 154.2288) (width 1.5) (layer "F.Cu") (net 8))
-  (segment (start 47.6504 151.3332) (end 45.212 151.3332) (width 1.5) (layer "F.Cu") (net 8))
+  (segment (start 46.228 127.7112) (end 42.8244 131.1148) (width 1.5) (layer "F.Cu") (net 8))
+  (segment (start 64.9224 117.0432) (end 64.9224 141.1224) (width 1.5) (layer "F.Cu") (net 8))
+  (segment (start 45.9232 151.3332) (end 42.8244 154.432) (width 1.5) (layer "F.Cu") (net 8))
   (segment (start 46.3296 151.3332) (end 47.6504 151.3332) (width 1.5) (layer "F.Cu") (net 8))
-  (segment (start 64.9224 117.0432) (end 64.9224 141.1224) (width 1.5) (layer "F.Cu") (net 8))
-  (segment (start 47.6504 127.7112) (end 45.72 127.7112) (width 1.5) (layer "F.Cu") (net 8))
+  (segment (start 46.7868 174.5488) (end 47.6504 174.5488) (width 1.5) (layer "F.Cu") (net 8))
+  (segment (start 42.8244 170.5864) (end 46.7868 174.5488) (width 1.5) (layer "F.Cu") (net 8))
   (segment (start 46.5836 127.7112) (end 45.0088 126.1364) (width 1.5) (layer "F.Cu") (net 8))
   (segment (start 45.0088 126.1364) (end 45.0088 108.7628) (width 1.5) (layer "F.Cu") (net 8))
   (segment (start 68.32872 144.52872) (end 87.62728 144.52872) (width 1.5) (layer "F.Cu") (net 8))
-  (segment (start 46.37136 174.5488) (end 47.6504 174.5488) (width 1.5) (layer "F.Cu") (net 8))
+  (segment (start 47.6504 127.7112) (end 46.228 127.7112) (width 1.5) (layer "F.Cu") (net 8))
   (segment (start 45.0088 108.7628) (end 46.482 107.2896) (width 1.5) (layer "F.Cu") (net 8))
-  (segment (start 42.8244 130.6068) (end 42.8244 147.828) (width 1.5) (layer "F.Cu") (net 8))
-  (segment (start 42.3164 170.49384) (end 46.37136 174.5488) (width 1.5) (layer "F.Cu") (net 8))
+  (segment (start 42.8244 154.432) (end 42.8244 170.5864) (width 1.5) (layer "F.Cu") (net 8))
+  (segment (start 42.8244 131.1148) (end 42.8244 147.828) (width 1.5) (layer "F.Cu") (net 8))
   (segment (start 55.1688 107.2896) (end 64.9224 117.0432) (width 1.5) (layer "F.Cu") (net 8))
-  (segment (start 42.3164 154.2288) (end 42.3164 170.49384) (width 1.5) (layer "F.Cu") (net 8))
   (segment (start 87.62728 144.52872) (end 87.7316 144.4244) (width 1.5) (layer "F.Cu") (net 8))
   (segment (start 42.8244 147.828) (end 46.3296 151.3332) (width 1.5) (layer "F.Cu") (net 8))
-  (segment (start 45.72 127.7112) (end 42.8244 130.6068) (width 1.5) (layer "F.Cu") (net 8))
   (segment (start 47.6504 172.0088) (end 51.0032 172.0088) (width 1.5) (layer "F.Cu") (net 9))
   (segment (start 47.6758 171.9834) (end 47.6504 172.0088) (width 0.75) (layer "F.Cu") (net 9))
@@
   (segment (start 47.6758 166.9034) (end 47.6504 166.9288) (width 0.75) (layer "F.Cu") (net 11))
   (segment (start 47.6504 166.9288) (end 51.0032 166.9288) (width 1.5) (layer "F.Cu") (net 11))
-  (segment (start 85.852 108.8136) (end 89.5604 108.8136) (width 1.5) (layer "F.Cu") (net 12))
-  (segment (start 91.0336 110.2868) (end 91.0336 159.9184) (width 1.5) (layer "F.Cu") (net 12))
+  (segment (start 45.20908 132.38772) (end 46.7868 130.81) (width 1.5) (layer "F.Cu") (net 12))
+  (segment (start 81.3308 113.3348) (end 85.852 108.8136) (width 1.5) (layer "F.Cu") (net 12))
+  (segment (start 85.852 108.8136) (end 89.7636 108.8136) (width 1.5) (layer "F.Cu") (net 12))
   (segment (start 56.0832 164.3888) (end 47.6504 164.3888) (width 1.5) (layer "F.Cu") (net 12))
-  (segment (start 45.20908 137.05548) (end 45.20908 132.66352) (width 1.5) (layer "F.Cu") (net 12))
+  (segment (start 89.7636 108.8136) (end 91.0336 110.0836) (width 1.5) (layer "F.Cu") (net 12))
   (segment (start 58.5724 142.91154) (end 56.83406 141.1732) (width 1.5) (layer "F.Cu") (net 12))
-  (segment (start 72.136 111.8616) (end 73.6092 113.3348) (width 1.5) (layer "F.Cu") (net 12))
+  (segment (start 45.20908 137.05548) (end 45.20908 132.38772) (width 1.5) (layer "F.Cu") (net 12))
   (segment (start 58.61092 171.99652) (end 58.6232 171.98424) (width 1.5) (layer "F.Cu") (net 12))
+  (segment (start 54.2187 130.81) (end 58.5724 126.4563) (width 1.5) (layer "F.Cu") (net 12))
   (segment (start 102.5508 181.5084) (end 102.5648 181.5224) (width 1.5) (layer "F.Cu") (net 12))
   (segment (start 77.76252 171.99652) (end 58.61092 171.99652) (width 1.5) (layer "F.Cu") (net 12))
@@
   (segment (start 82.8764 181.356) (end 82.8548 181.3344) (width 1.5) (layer "F.Cu") (net 12))
   (segment (start 70.3072 103.6828) (end 98.552 103.6828) (width 1.5) (layer "F.Cu") (net 12))
+  (segment (start 73.6092 113.3348) (end 81.3308 113.3348) (width 1.5) (layer "F.Cu") (net 12))
   (segment (start 46.0756 161.8488) (end 45.212 160.9852) (width 1.5) (layer "F.Cu") (net 12))
+  (segment (start 46.7868 138.6332) (end 45.20908 137.05548) (width 1.5) (layer "F.Cu") (net 12))
   (segment (start 69.1388 131.6736) (end 74.5744 131.6736) (width 1.5) (layer "F.Cu") (net 12))
-  (segment (start 81.3308 113.3348) (end 85.852 108.8136) (width 1.5) (layer "F.Cu") (net 12))
   (segment (start 47.6504 138.6332) (end 47.6504 141.1732) (width 1.5) (layer "F.Cu") (net 12))
   (segment (start 88.75032 162.20168) (end 87.72792 162.20168) (width 1.5) (layer "F.Cu") (net 12))
   (segment (start 82.8764 177.1104) (end 77.76252 171.99652) (width 1.5) (layer "F.Cu") (net 12))
   (segment (start 98.552 103.6828) (end 103.5812 108.712) (width 1.5) (layer "F.Cu") (net 12))
-  (segment (start 47.6504 138.6332) (end 46.7868 138.6332) (width 1.5) (layer "F.Cu") (net 12))
   (segment (start 58.6232 166.9288) (end 56.0832 164.3888) (width 1.5) (layer "F.Cu") (net 12))
   (segment (start 77.342 128.906) (end 78.9824 128.906) (width 1.5) (layer "F.Cu") (net 12))
@@
   (segment (start 58.5724 143.8148) (end 58.5724 142.91154) (width 1.5) (layer "F.Cu") (net 12))
   (segment (start 57.44366 117.5512) (end 47.6504 117.5512) (width 1.5) (layer "F.Cu") (net 12))
-  (segment (start 73.6092 113.3348) (end 81.3308 113.3348) (width 1.5) (layer "F.Cu") (net 12))
-  (segment (start 53.70798 131.32072) (end 58.5724 126.4563) (width 1.5) (layer "F.Cu") (net 12))
   (segment (start 58.5724 149.9259) (end 58.5724 148.8948) (width 1.5) (layer "F.Cu") (net 12))
   (segment (start 46.86028 153.74892) (end 54.74938 153.74892) (width 1.5) (layer "F.Cu") (net 12))
   (segment (start 58.5724 120.0912) (end 58.5724 118.67994) (width 1.5) (layer "F.Cu") (net 12))
+  (segment (start 58.5724 126.4563) (end 58.5724 125.1712) (width 1.5) (layer "F.Cu") (net 12))
   (segment (start 107.3404 167.0812) (end 114.1476 167.0812) (width 1.5) (layer "F.Cu") (net 12))
   (segment (start 47.6504 161.8488) (end 46.0756 161.8488) (width 1.5) (layer "F.Cu") (net 12))
   (segment (start 93.9292 181.4824) (end 93.9032 181.5084) (width 1.5) (layer "F.Cu") (net 12))
   (segment (start 103.5812 163.322) (end 107.3404 167.0812) (width 1.5) (layer "F.Cu") (net 12))
-  (segment (start 89.5604 108.8136) (end 91.0336 110.2868) (width 1.5) (layer "F.Cu") (net 12))
+  (segment (start 46.7868 130.81) (end 54.2187 130.81) (width 1.5) (layer "F.Cu") (net 12))
   (segment (start 67.1576 106.8324) (end 70.3072 103.6828) (width 1.5) (layer "F.Cu") (net 12))
   (segment (start 45.212 160.9852) (end 45.212 155.3972) (width 1.5) (layer "F.Cu") (net 12))
@@
   (segment (start 58.5724 125.1712) (end 58.5724 122.6312) (width 1.5) (layer "F.Cu") (net 12))
   (segment (start 103.5812 108.712) (end 103.5812 163.322) (width 1.5) (layer "F.Cu") (net 12))
+  (segment (start 47.6504 138.6332) (end 46.7868 138.6332) (width 1.5) (layer "F.Cu") (net 12))
   (segment (start 58.5724 118.67994) (end 57.44366 117.5512) (width 1.5) (layer "F.Cu") (net 12))
+  (segment (start 91.0336 159.9184) (end 88.75032 162.20168) (width 1.5) (layer "F.Cu") (net 12))
   (segment (start 82.8548 181.3344) (end 82.8548 166.624) (width 1.5) (layer "F.Cu") (net 12))
   (segment (start 82.8764 181.356) (end 82.8764 177.1104) (width 1.5) (layer "F.Cu") (net 12))
-  (segment (start 91.0336 159.9184) (end 88.75032 162.20168) (width 1.5) (layer "F.Cu") (net 12))
   (segment (start 47.6504 115.0112) (end 47.6504 117.5512) (width 1.5) (layer "F.Cu") (net 12))
   (segment (start 58.5724 148.8948) (end 58.5724 146.3548) (width 1.5) (layer "F.Cu") (net 12))
-  (segment (start 45.20908 132.66352) (end 46.55188 131.32072) (width 1.5) (layer "F.Cu") (net 12))
-  (segment (start 58.5724 126.4563) (end 58.5724 125.1712) (width 1.5) (layer "F.Cu") (net 12))
+  (segment (start 72.136 111.8616) (end 73.6092 113.3348) (width 1.5) (layer "F.Cu") (net 12))
+  (segment (start 91.0336 110.0836) (end 91.0336 159.9184) (width 1.5) (layer "F.Cu") (net 12))
   (segment (start 67.1576 129.9464) (end 67.1576 106.8324) (width 1.5) (layer "F.Cu") (net 12))
   (segment (start 58.5724 146.3548) (end 58.5724 143.8148) (width 1.5) (layer "F.Cu") (net 12))
   (segment (start 114.1476 167.0812) (end 114.0968 167.0812) (width 0.75) (layer "F.Cu") (net 12))
-  (segment (start 46.7868 138.6332) (end 45.20908 137.05548) (width 1.5) (layer "F.Cu") (net 12))
   (segment (start 54.74938 153.74892) (end 58.5724 149.9259) (width 1.5) (layer "F.Cu") (net 12))
   (segment (start 93.9032 181.5084) (end 83.0288 181.5084) (width 1.5) (layer "F.Cu") (net 12))
   (segment (start 58.6232 171.98424) (end 58.6232 166.9288) (width 1.5) (layer "F.Cu") (net 12))
-  (segment (start 46.55188 131.32072) (end 53.70798 131.32072) (width 1.5) (layer "F.Cu") (net 12))
   (segment (start 104.2924 167.0812) (end 114.1476 167.0812) (width 1.5) (layer "B.Cu") (net 12))
   (segment (start 99.41288 162.20168) (end 104.2924 167.0812) (width 1.5) (layer "B.Cu") (net 12))
