File: MainBoardV3/MainboardV3.kicad_sch (KiCad schematic)
At the start: 44 parts, among them J10 Conn_01x04, J11 Conn_01x02, J12 Conn_01x03, J13 Conn_01x03, J14 Conn_01x03, J15 Conn_01x03, J16 Conn_01x02, J17 Conn_01x02, J18 Conn_01x03, J19 Conn_01x03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

Commit message: La V3 en mode, je ne sais quoi
Parts:
- removed C1, C2: C_Small, Capacitor_SMD:C_0805_2012Metric_Pad1.18x1.45mm_HandSolder, symbol Device:C_Small
- removed D2: WS2812B, LED_SMD:LED_WS2812B_PLCC4_5.0x5.0mm_P3.2mm, symbol LED:WS2812B
- removed D4: LED_Small, LED_SMD:LED_1206_3216Metric_Pad1.42x1.75mm_HandSolder, symbol Device:LED_Small
- removed J12, J13, J14, J15, J19, J20, J21: Conn_01x03, Connector_PinHeader_2.54mm:PinHeader_1x03_P2.54mm_Vertical, symbol Connector_Generic:Conn_01x03
- removed J16, J17: Conn_01x02, Connector_PinHeader_2.54mm:PinHeader_1x02_P2.54mm_Vertical, symbol Connector_Generic:Conn_01x02
- removed R5: R_Small, Resistor_SMD:R_1206_3216Metric_Pad1.30x1.75mm_HandSolder, symbol Device:R_Small
- removed SW3, SW4, SW5: SW_DIP_x03, Button_Switch_THT:SW_DIP_SPSTx03_Slide_9.78x9.8mm_W7.62mm_P2.54mm, symbol Switch:SW_DIP_x03
- removed U1: AMS1117-3.3, Package_TO_SOT_SMD:SOT-223-3_TabPin2, symbol Regulator_Linear:AMS1117-3.3
- added J1: Conn_01x02, Connector_JST:JST_XH_B2B-XH-A_1x02_P2.50mm_Vertical, symbol Connector_Generic:Conn_01x02
- added J19, J20, J21: Conn_02x03_Odd_Even, Connector_PinHeader_2.54mm:PinHeader_2x03_P2.54mm_Vertical, symbol Connector_Generic:Conn_02x03_Odd_Even
- added J24: Conn_02x05_Odd_Even, Connector_IDC:IDC-Header_2x05_P2.54mm_Vertical, symbol Connector_Generic:Conn_02x05_Odd_Even
- J11: footprint Connector_PinHeader_2.54mm:PinHeader_1x02_P2.54mm_Vertical -> Connector_JST:JST_XH_B2B-XH-A_1x02_P2.50mm_Vertical
- R1: footprint Resistor_THT:R_Axial_DIN0204_L3.6mm_D1.6mm_P5.08mm_Vertical -> Resistor_SMD:R_1206_3216Metric_Pad1.30x1.75mm_HandSolder
- R2: footprint Resistor_THT:R_Axial_DIN0204_L3.6mm_D1.6mm_P7.62mm_Horizontal -> Resistor_SMD:R_1206_3216Metric_Pad1.30x1.75mm_HandSolder
- U2: footprint ESP32:ESP32-S3-DevKitC -> ESP:ESP32-S3-DevKitC
Connections:
- net +5V: now also J3.1 (Pin_1), J19.1 (Pin_1), J19.3 (Pin_3), J19.5 (Pin_5), J20.1 (Pin_1), J20.3 (Pin_3), J20.5 (Pin_5), J21.1 (Pin_1), J21.3 (Pin_3), J21.5 (Pin_5)
- net GND: now also J11.2 (Pin_2), J3.3 (Pin_3), J1.2 (Pin_2), J24.1 (Pin_1); no longer J3.1 (Pin_1)
- net GP2: now also J1.1 (Pin_1); no longer J11.2 (Pin_2)
- net Neopixel: now also J3.2 (Pin_2)
- net at A3.12 (M2): now also J21.6 (Pin_6)
- net at A3.11 (M1): now also J21.4 (Pin_4)
- net at A3.10 (M0): now also J21.2 (Pin_2)
- net at A2.10 (M0): now also J20.2 (Pin_2)
- net at A2.11 (M1): now also J20.4 (Pin_4)
- net at A2.12 (M2): now also J20.6 (Pin_6)
- net at A1.10 (M0): now also J19.2 (Pin_2)
- net at A1.11 (M1): now also J19.4 (Pin_4)
- net at A1.12 (M2): now also J19.6 (Pin_6)
- net GP35: no longer names the net of U2.32 (GPIO35)
- net GP36: no longer names the net of U2.33 (GPIO36)
- net GP37: no longer names the net of U2.34 (GPIO37)
- net GP38: no longer names the net of U2.35 (GPIO38)
- net GP38: no longer J3.3 (Pin_3)
- no-connect marks 9 -> 8
Other:
- sheet Power: file Power.kicad_sch -> Power sheet.kicad_sch
- sheet Power ports: added PwrEn; removed none
- moved on the sheet: H1, J11

Commit message: Mise a jour pour remi
Parts:
- added U5: ~, Custom:PCA9685breakout, symbol PCM:PWMI2C
- H1, H2, H3, H4: footprint MountingHole:MountingHole_3.2mm_M3_DIN965_Pad -> MountingHole:MountingHole_3.2mm_M3
Connections:
- net +5V: now also J3.2 (Pin_2), U5.4 (VCC); no longer J3.1 (Pin_1)
- net GND: now also J24.10 (Pin_10), U5.0 (GND)
- net Neopixel: now also J3.1 (Pin_1); no longer J3.2 (Pin_2)
- net SCL: now also U5.2 (SCL)
- net SDA: now also U5.3 (SDA)
- net GPIO21: now reaches J24.2 (Pin_2)
- net GPIO21: now also U2.27 (GPIO21)
- net GPIO38: now reaches J24.3 (Pin_3)
- net GPIO38: now also U2.35 (GPIO38)
- net GPIO47: now reaches J24.4 (Pin_4)
- net GPIO47: now also U2.28 (GPIO47)
- net GPIO37: now reaches J24.5 (Pin_5)
- net GPIO37: now also U2.34 (GPIO37)
- net GPIO48: now reaches J24.6 (Pin_6)
- net GPIO48: now also U2.29 (GPIO48)
- net GPIO36: now reaches J24.7 (Pin_7)
- net GPIO36: now also U2.33 (GPIO36)
- net GPIO45: now reaches J24.8 (Pin_8)
- net GPIO45: now also U2.30 (GPIO45)
- net GPI035: now reaches J24.9 (Pin_9)
- net GPI035: now also U2.32 (GPIO35)
- new net +5VP: U5.5 (V+_6VMax)
Other:
- moved on the sheet: H3, J24
