File: MainBoardV3/Power sheet.kicad_sch (KiCad schematic)
At the start: 22 parts, among them J12 Conn_01x02, J13 Conn_01x02, J14 Conn_01x02, J15 Conn_01x02, J16 Conn_01x02, J17 Conn_01x02, J6 Conn_01x02, U1 TSR_2-2450, U3 TSR_2-2433, U4 TEN_50-2411WI

Commit message: Mise a jour pour remi
Parts:
- removed C6: C_Polarized, symbol Device:C_Polarized
- C1, C2, C4: footprint (none) -> Capacitor_THT:CP_Radial_D5.0mm_P2.50mm
- C3: footprint (none) -> Capacitor_THT:CP_Radial_D8.0mm_P3.80mm
- C5: footprint (none) -> Capacitor_THT:CP_Radial_D8.0mm_P3.50mm
Other:
- moved on the sheet: C1, C4, C5, D4, J6, R5, U3, U4

Commit message: V0.4 modifications all components attached
Connections:
- net +12V: now also J6.2 (Pin_2); no longer J6.1 (Pin_1)
- net GND: now also J6.1 (Pin_1); no longer J6.2 (Pin_2)
Changed lines of the file:
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@@
-    )
-  )
-  (symbol (lib_id "Connector_Generic:Conn_01x02") (at 146.685 136.525 0) (unit 1)
-    (in_bom yes) (on_board yes) (dnp no) (fields_autoplaced)
-    (property "Reference" "J6" (at 149.225 136.525 0)
-      (effects (font (size 1.27 1.27)) (justify left))
-    )
-    (property "Value" "Conn_01x02" (at 149.225 139.065 0)
-      (effects (font (size 1.27 1.27)) (justify left))
-    )
-    (property "Footprint" "Connector_AMASS:AMASS_XT60-M_1x02_P7.20mm_Vertical" (at 146.685 136.525 0)
-      (effects (font (size 1.27 1.27)) hide)
-    )
-    (property "Datasheet" "~" (at 146.685 136.525 0)
-      (effects (font (size 1.27 1.27)) hide)
-    )
-    (pin "1")
-    (pin "2")
-    (instances
-      (project "MainboardV3"
-        (path "/ccdda621-e361-4147-9a57-71374655ba08/cc39ea4c-864b-49b2-93dc-48ce7f75ef7f"
-          (reference "J6") (unit 1)
-        )
-      )
     )
   )
@@
         )
       )
+    )
+  )
+  (symbol (lib_id "Connector_Generic:Conn_01x02") (at 146.685 139.065 0) (mirror x) (unit 1)
+    (in_bom yes) (on_board yes) (dnp no)
+    (property "Reference" "J6" (at 149.225 139.065 0)
+      (effects (font (size 1.27 1.27)) (justify left))
+    )
+    (property "Value" "Conn_01x02" (at 149.225 136.525 0)
+      (effects (font (size 1.27 1.27)) (justify left))
+    )
+    (property "Footprint" "Connector_AMASS:AMASS_XT60-M_1x02_P7.20mm_Vertical" (at 146.685 139.065 0)
+      (effects (font (size 1.27 1.27)) hide)
+    )
+    (property "Datasheet" "~" (at 146.685 139.065 0)
+      (effects (font (size 1.27 1.27)) hide)
+    )
+    (pin "1")
+    (pin "2")
+    (instances
+      (project "MainboardV3"
+        (path "/ccdda621-e361-4147-9a57-71374655ba08/cc39ea4c-864b-49b2-93dc-48ce7f75ef7f"
+          (reference "J6") (unit 1)
+        )
+      )
