File: MainBoardV3/MainboardV3.kicad_pcb (KiCad board)
At the start: 2 copper layers, 50 parts, among them J1 Conn_01x02, J10 Conn_01x04, J11 Conn_01x02, J12 Conn_01x03, J13 Conn_01x03, J14 Conn_01x03, J15 Conn_01x03, J16 Conn_01x02, J17 Conn_01x02, J18 Conn_01x03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

Commit message: La V3 en mode, je ne sais quoi
Parts:
- removed C1, C2: C_Small, Capacitor_SMD:C_0805_2012Metric_Pad1.18x1.45mm_HandSolder
- removed D2: WS2812B, LED_SMD:LED_WS2812B_PLCC4_5.0x5.0mm_P3.2mm
- removed SW3, SW4, SW5: SW_DIP_x03, Button_Switch_THT:SW_DIP_SPSTx03_Slide_9.78x9.8mm_W7.62mm_P2.54mm
- added J24: Conn_02x05_Odd_Even, Connector_IDC:IDC-Header_2x05_P2.54mm_Vertical, F.Cu at (42.6, -4.83)
- added U3: TSR_2-2433, Traco:Traco 2- 24xx, F.Cu at (-29.5, 32.6)
- added U4: TEN_50-2411WI, Traco:Traco TEN 50 series, F.Cu at (4.83, 34.3)
- J1: footprint TerminalBlock:TerminalBlock_Altech_AK300-2_P5.00mm -> Connector_JST:JST_XH_B2B-XH-A_1x02_P2.50mm_Vertical
- J11: footprint Connector_PinHeader_2.54mm:PinHeader_1x02_P2.54mm_Vertical -> Connector_JST:JST_XH_B2B-XH-A_1x02_P2.50mm_Vertical
- J12, J13, J14, J15: value Conn_01x03 -> Conn_01x02; footprint Connector_PinHeader_2.54mm:PinHeader_1x03_P2.54mm_Vertical -> Connector_Molex:Molex_KK-254_AE-6410-02A_1x02_P2.54mm_Vertical
- J16, J17: footprint Connector_PinHeader_2.54mm:PinHeader_1x02_P2.54mm_Vertical -> Connector_Molex:Molex_KK-254_AE-6410-02A_1x02_P2.54mm_Vertical
- J19, J20, J21: value Conn_01x03 -> Conn_02x03_Odd_Even; footprint Connector_PinHeader_2.54mm:PinHeader_1x03_P2.54mm_Vertical -> Connector_PinHeader_2.54mm:PinHeader_2x03_P2.54mm_Vertical
- J5: moved to B.Cu
- J6: footprint TerminalBlock:TerminalBlock_Altech_AK300-2_P5.00mm -> Connector_AMASS:AMASS_XT60-M_1x02_P7.20mm_Vertical
- R1: footprint Resistor_THT:R_Axial_DIN0204_L3.6mm_D1.6mm_P5.08mm_Vertical -> Resistor_SMD:R_1206_3216Metric_Pad1.30x1.75mm_HandSolder
- R2: footprint Resistor_THT:R_Axial_DIN0204_L3.6mm_D1.6mm_P7.62mm_Horizontal -> Resistor_SMD:R_1206_3216Metric_Pad1.30x1.75mm_HandSolder
- U1: value AMS1117-3.3 -> TSR_2-2450; footprint Package_TO_SOT_SMD:SOT-223-3_TabPin2 -> Traco:Traco 2- 24xx
- U2: footprint ESP32:ESP32-S3-DevKitC -> ESP:ESP32-S3-DevKitC
- moved H4 134.9 mm to (-46.5, -45.9)
- moved J1 126.3 mm to (39.0, -35.8), turned to 90 degrees
- moved R3 119.4 mm to (-30.7, 38.3)
- moved R4 119.1 mm to (-30.6, 40.9)
- moved J9 117.5 mm to (-13.5, -40.5), turned to -90 degrees
- moved R1 110.7 mm to (17.3, -37.7)
- moved J5 109.4 mm to (-9.97, -25.2), turned to -90 degrees
- moved D1 108.3 mm to (-25.1, 38.4), turned to 180 degrees
- moved D3 108.0 mm to (-25.1, 41.0), turned to 180 degrees
- moved J8 106.9 mm to (-5.97, -40.6), turned to -90 degrees
- moved J23 105.8 mm to (46.9, -35.5), turned to -90 degrees
- moved H3 100.3 mm to (46.5, -46.5)
- moved J7 96.2 mm to (1.52, -40.5), turned to -90 degrees
- moved J21 95.7 mm to (-20.5, -30.5), turned to 180 degrees
- moved C7 93.9 mm to (-45.6, -24.6)
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Connections:
- J1 pad 1: +12V -> /GP2
- J11 pad 2: /GP2 -> GND
- J12 pad 1: GND -> +12V
- J12 pad 2: Net-(J12-Pin_2) -> GND
- J13 pad 1: GND -> +12V
- J13 pad 2: Net-(J12-Pin_2) -> GND
- J14 pad 1: GND -> +12V
- J14 pad 2: Net-(J12-Pin_2) -> GND
- J15 pad 1: +3.3VP -> +5VP
- J15 pad 2: Net-(J12-Pin_2) -> GND
- J16 pad 1: +12V -> +5VP
- J16 pad 2: +12V -> GND
- J17 pad 1: GND -> +5VP
- J19 pad 1: GND -> +5V
- J19 pad 2: Net-(J12-Pin_2) -> Net-(A1-M0)
- J19 pad 3: Net-(J19-Pin_3) -> +5V
- J20 pad 1: GND -> +5V
- J20 pad 2: Net-(J12-Pin_2) -> Net-(A2-M0)
- J20 pad 3: Net-(J20-Pin_3) -> +5V
- J21 pad 1: GND -> +5V
- J21 pad 2: Net-(J12-Pin_2) -> Net-(A3-M0)
- J21 pad 3: Net-(J21-Pin_3) -> +5V
- J3 pad 1: GND -> +5V
- J3 pad 2: Net-(J12-Pin_2) -> Neopixel
- J3 pad 3: /GP38 -> GND
- J6 pad 1: GND -> +12V
- J6 pad 2: +5V -> GND
- R3 pad 1: +5V -> +3.3VP
- R4 pad 1: Net-(D3-A) -> +5V
- R4 pad 2: +12V -> Net-(D3-A)
- R5 pad 1: +3.3VP -> +12V
- U1 pad 1: GND -> +12V
- U1 pad 2: +3.3VP -> GND
- U2 pad 28: Net-(J20-Pin_3) -> unconnected-(U2-GPIO47-Pad28)
- U2 pad 29: Net-(J21-Pin_3) -> unconnected-(U2-GPIO48-Pad29)
- U2 pad 30: Net-(J19-Pin_3) -> unconnected-(U2-GPIO45-Pad30)
- U2 pad 32: /GP35 -> unconnected-(U2-GPIO35-Pad32)
- U2 pad 33: /GP36 -> unconnected-(U2-GPIO36-Pad33)
- U2 pad 34: /GP37 -> unconnected-(U2-GPIO37-Pad34)
- U2 pad 35: /GP38 -> unconnected-(U2-GPIO38-Pad35)
Other:
- board outline added: 100 x 100 mm

Commit message: Mise a jour pour remi
Parts:
- added C1: C_Polarized, Capacitor_THT:CP_Radial_D5.0mm_P2.50mm, F.Cu at (7.75, 48.0)
- added C2: C_Polarized, Capacitor_THT:CP_Radial_D5.0mm_P2.50mm, F.Cu at (25.5, 32.5)
- added C3: C_Polarized, Capacitor_THT:CP_Radial_D8.0mm_P3.80mm, F.Cu at (-26.8, 47.2)
- added C4: C_Polarized, Capacitor_THT:CP_Radial_D5.0mm_P2.50mm, F.Cu at (17.5, 32.2)
- added C5: C_Polarized, Capacitor_THT:CP_Radial_D8.0mm_P3.50mm, F.Cu at (10.2, 39.6)
- added U5: ~, Custom:PCA9685breakout, F.Cu at (65.2, 13.4)
- H1, H2, H3, H4: footprint MountingHole:MountingHole_3.2mm_M3_DIN965_Pad -> MountingHole:MountingHole_3.2mm_M3
- J19, J8: moved to B.Cu
- moved J18 88.0 mm to (-13.5, -46.0), turned to 0 degrees
- moved U1 57.5 mm to (25.0, 42.5), turned to 90 degrees
- moved R3 51.0 mm to (18.3, 24.2)
- moved R4 51.0 mm to (18.3, 26.8)
- moved D1 50.7 mm to (23.6, 24.3)
- moved D3 50.7 mm to (23.6, 26.8)
- moved U3 47.3 mm to (16.8, 42.5), turned to 90 degrees
- moved J16 27.7 mm to (9.02, 24.7), turned to 180 degrees
- moved J17 27.7 mm to (9.00, 17.8), turned to 180 degrees
- moved J15 27.7 mm to (9.02, 31.7), turned to 180 degrees
- moved J12 27.3 mm to (-26.3, 23.2)
- moved J13 17.7 mm to (-26.3, 30.2)
- moved U4 16.8 mm to (-8.50, 24.0), turned to 90 degrees
- moved J19 13.0 mm to (-30.2, 24.0), turned to 90 degrees
- moved R2 10.8 mm to (17.0, -29.9), turned to 180 degrees
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Connections:
- J24 pad 10: unconnected-(J24-Pin_10-Pad10) -> GND
- J24 pad 2: unconnected-(J24-Pin_2-Pad2) -> GPIO21
- J24 pad 3: unconnected-(J24-Pin_3-Pad3) -> GPIO38
- J24 pad 4: unconnected-(J24-Pin_4-Pad4) -> GPIO47
- J24 pad 5: unconnected-(J24-Pin_5-Pad5) -> GPIO37
- J24 pad 6: unconnected-(J24-Pin_6-Pad6) -> GPIO48
- J24 pad 7: unconnected-(J24-Pin_7-Pad7) -> GPIO36
- J24 pad 8: unconnected-(J24-Pin_8-Pad8) -> GPIO45
- J24 pad 9: unconnected-(J24-Pin_9-Pad9) -> GPI035
- J3 pad 1: +5V -> Neopixel
- J3 pad 2: Neopixel -> +5V
- U2 pad 27: unconnected-(U2-GPIO21-Pad27) -> GPIO21
- U2 pad 28: unconnected-(U2-GPIO47-Pad28) -> GPIO47
- U2 pad 29: unconnected-(U2-GPIO48-Pad29) -> GPIO48
- U2 pad 30: unconnected-(U2-GPIO45-Pad30) -> GPIO45
- U2 pad 32: unconnected-(U2-GPIO35-Pad32) -> GPI035
- U2 pad 33: unconnected-(U2-GPIO36-Pad33) -> GPIO36
- U2 pad 34: unconnected-(U2-GPIO37-Pad34) -> GPIO37
- U2 pad 35: unconnected-(U2-GPIO38-Pad35) -> GPIO38
Routing:
- net +5V: track 0.00 -> 284.4 mm
- net +12V: track 0.00 -> 214.2 mm
- net EN: track 0.00 -> 135.2 mm
- net +3.3VP: track 0.00 -> 116.5 mm, vias 0 -> 1
- net SDA: track 0.00 -> 87.0 mm
- net SCL: track 0.00 -> 86.9 mm
- net +5VP: track 0.00 -> 70.2 mm
- net STEP3: track 0.00 -> 58.3 mm
- net DIR3: track 0.00 -> 58.2 mm
- net STEP2: track 0.00 -> 39.7 mm
- net DIR2: track 0.00 -> 39.7 mm
- net STEP1: track 0.00 -> 36.9 mm
- net DIR1: track 0.00 -> 36.2 mm
- net +3.3V: track 0.00 -> 24.5 mm
- net GND: track 0.00 -> 18.6 mm, vias 0 -> 3
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- added copper zone on B.Cu, net GND
- added copper zone on F.Cu, net GND
Other:
- board text added: "Unimakers CDR 2024 Looij Dylan V0.3"

Commit message: V0.4 modifications all components attached
Parts:
- moved J6 7.15 mm to (-44.3, 29.8), turned to -90 degrees
- moved U1 1.80 mm to (26.8, 42.6)
- moved U3 1.35 mm to (18.1, 42.6)
- moved J17 0.70 mm to (9.70, 17.8)
- moved J15 0.69 mm to (9.70, 31.6)
- moved J16 0.68 mm to (9.70, 24.7)
- moved C5 0.32 mm to (10.5, 39.5)
Connections:
- J6 pad 1: +12V -> GND
- J6 pad 2: GND -> +12V
Routing:
- net GPIO38: track 0.00 -> 34.2 mm
- net GPIO37: track 0.00 -> 27.5 mm
- net GPIO36: track 0.00 -> 20.7 mm
- net GPI035: track 0.00 -> 13.5 mm
- net +12V: track 214.2 -> 215.9 mm
- net +5VP: track 70.2 -> 69.5 mm
- net +5V: track 284.4 -> 285.0 mm

Commit message: test
Changed lines of the file:
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@@
     (pad "" np_thru_hole circle (at 27.813 -9.398) (size 1.524 1.524) (drill 2.5) (layers "F&B.Cu" "*.Mask"))
     (pad "" np_thru_hole circle (at 27.813 9.398) (size 1.524 1.524) (drill 2.5) (layers "F&B.Cu" "*.Mask"))
-    (pad "0" thru_hole circle (at -29.083 -6.35) (size 1.524 1.524) (drill 0.6) (layers "*.Cu" "*.Mask")
+    (pad "0" thru_hole circle (at -29.083 -6.35) (size 1.524 1.524) (drill 0.762) (layers "*.Cu" "*.Mask")
       (net 1 "GND") (pinfunction "GND") (pintype "input"))
-    (pad "0" thru_hole circle (at 29.083 -6.35) (size 1.524 1.524) (drill 0.6) (layers "*.Cu" "*.Mask")
+    (pad "0" thru_hole circle (at 29.083 -6.35) (size 1.524 1.524) (drill 0.762) (layers "*.Cu" "*.Mask")
       (net 1 "GND") (pinfunction "GND") (pintype "input"))
     (pad "1" thru_hole circle (at -29.083 -3.81) (size 1.524 1.524) (drill 0.762) (layers "*.Cu" "*.Mask")
