File: MainBoardV4/MainBoardV4.kicad_pcb (KiCad board)
At the start: 2 copper layers, 100 x 100 mm, 85 parts, among them J1 Conn_01x02, J11 Conn_01x03, J12 USB_B_Micro, J13 Conn_02x03_Odd_Even, J14 Conn_01x04, J15 Conn_02x03_Odd_Even, J16 Conn_01x04, J17 Conn_02x03_Odd_Even, J18 Conn_01x04, J19 Conn_01x04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

Commit message: test
Routing:
- net SCL: track 73.4 -> 80.1 mm
- net Net-(RN5-R3.1): track 5.10 -> 4.40 mm
- net Net-(RN6-R3.1): track 10.9 -> 11.6 mm
- net Net-(RN5-R2.1): track 6.51 -> 5.92 mm
