File: MainBoardV1/MainBoardV1.kicad_sch (KiCad schematic)
At the start: 32 parts, among them J1 USB_B_Micro, J10 Conn_01x04, J2 Conn_01x04, J3 Conn_01x02, J4 Conn_01x04, J5 Conn_01x05, J6 Conn_01x02, J7 Conn_01x04, J8 Conn_01x04, J9 Conn_01x04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

Commit message: Merge of versions
Other:
- moved on the sheet: A1, A2, A3, C1, C2, C3, C4, C5, C6, C7, C8, C9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
